Commit message: urdf, gazebo files added

File: robotis_arm/urdf/gazebo_preparing.urdf (robot description, URDF)
Before this commit: robot model, 16 links, 15 joints
Links:
- link base_link: mass None -> 10; geometry collision cylinder lenght=0.6 radius=0.2; visual cylinder length=0.6 radius=0.2
- link box: mass None -> 10; geometry collision box size=0.08 0.08 0.08; visual box size=0.08 0.08 0.08
- link gripper_pole: mass None -> 0.05; geometry collision cylinder length=0.2 radius=0.01; visual cylinder length=0.2 radius=0.01
- link head: mass None -> 2; geometry collision sphere radius=0.2; visual sphere radius=0.2
- link left_back_wheel: mass None -> 1; geometry collision cylinder length=0.1 radius=0.035; visual cylinder length=0.1 radius=0.035
- link left_base: mass None -> 10; geometry collision box size=0.4 0.1 0.1; visual box size=0.4 0.1 0.1
- link left_front_wheel: mass None -> 1; geometry collision cylinder length=0.1 radius=0.035; visual cylinder length=0.1 radius=0.035
- link left_gripper: mass None -> 0.05; geometry collision mesh filename=package://urdf_tutorial/meshes/l_finger.dae; visual mesh filename=package://urdf_tutorial/meshes/l_finger.dae
- link left_leg: mass None -> 10; geometry collision box size=0.6 0.1 0.2; visual box size=0.6 0.1 0.2
- link left_tip: mass None -> 0.05; geometry collision mesh filename=package://urdf_tutorial/meshes/l_finger_tip.dae; visual mesh filename=package://urdf_tutorial/meshes/l_finger_tip.dae
- link right_back_wheel: mass None -> 1; geometry collision cylinder length=0.1 radius=0.035; visual cylinder length=0.1 radius=0.035
- link right_base: mass None -> 10; geometry collision box size=0.4 0.1 0.1; visual box size=0.4 0.1 0.1
- link right_front_wheel: mass None -> 1; geometry collision cylinder length=0.1 radius=0.035; visual cylinder length=0.1 radius=0.035
- link right_gripper: mass None -> 0.05; geometry collision mesh filename=package://urdf_tutorial/meshes/l_finger.dae; visual mesh filename=package://urdf_tutorial/meshes/l_finger.dae
- link right_leg: mass None -> 10; geometry collision box size=0.6 0.1 0.2; visual box size=0.6 0.1 0.2
- link right_tip: mass None -> 0.05; geometry collision mesh filename=package://urdf_tutorial/meshes/l_finger_tip.dae; visual mesh filename=package://urdf_tutorial/meshes/l_finger_tip.dae
