Commit message: controller edited

File: robotic_arm/urdf/open_manipulator.gazebo.xacro (robot description, xacro)
@@ -1,92 +1,181 @@
 <?xml version="1.0"?>
-<robot xmlns:xacro="http://ros.org/wiki/xacro">
-  <!-- Gazebo Reference macro -->
-  <xacro:macro name="RefLink" params="ref">
-    <gazebo reference="${ref}">
-      <kp>1000000.0</kp>
-      <kd>100.0</kd>
-      <mu1>30.0</mu1>
-      <mu2>30.0</mu2>
-      <maxVel>1.0</maxVel>
-      <minDepth>0.001</minDepth>
-      <material>Gazebo/DarkGrey</material>
-    </gazebo>
-  </xacro:macro>
+<robot>
   <!-- World -->
-  <gazebo reference="world"/>
+  <gazebo reference="world">
+  </gazebo>
   <!-- Link1 -->
-  <RefLink ref="link1"/>
+  <gazebo reference="link1">
+    <kp>1000000.0</kp>
+    <kd>100.0</kd>
+    <mu1>30.0</mu1>
+    <mu2>30.0</mu2>
+    <maxVel>1.0</maxVel>
+    <minDepth>0.001</minDepth>
+    <material>Gazebo/DarkGrey</material>
+  </gazebo>
   <!-- Link2 -->
-  <RefLink ref="link2"/>
+  <gazebo reference="link2">
+    <kp>1000000.0</kp>
+    <kd>100.0</kd>
+    <mu1>30.0</mu1>
+    <mu2>30.0</mu2>
+    <maxVel>1.0</maxVel>
+    <minDepth>0.001</minDepth>
+    <material>Gazebo/DarkGrey</material>
+  </gazebo>
   <!-- Link3 -->
-  <RefLink ref="link3"/>
+  <gazebo reference="link3">
+    <kp>1000000.0</kp>
+    <kd>100.0</kd>
+    <mu1>30.0</mu1>
+    <mu2>30.0</mu2>
+    <maxVel>1.0</maxVel>
+    <minDepth>0.001</minDepth>
+    <material>Gazebo/DarkGrey</material>
+  </gazebo>
   <!-- Link4 -->
-  <RefLink ref="link4"/>
+  <gazebo reference="link4">
+    <kp>1000000.0</kp>
+    <kd>100.0</kd>
+    <mu1>30.0</mu1>
+    <mu2>30.0</mu2>
+    <maxVel>1.0</maxVel>
+    <minDepth>0.001</minDepth>
+    <material>Gazebo/DarkGrey</material>
+  </gazebo>
   <!-- Link5 -->
-  <RefLink ref="link5"/>
-  <!-- gripper_link -->
-  <RefLink ref="gripper_link"/>
-  <!-- gripper_link_sub -->
-  <RefLink ref="gripper_link_sub"/>
-  <!-- end effector link -->
-  <gazebo reference="end_effector_link">
-    <material>Gazebo/Red</material>
+  <gazebo reference="link5">
+    <kp>1000000.0</kp>
+    <kd>100.0</kd>
+    <mu1>30.0</mu1>
+    <mu2>30.0</mu2>
+    <maxVel>1.0</maxVel>
+    <minDepth>0.001</minDepth>
+    <material>Gazebo/DarkGrey</material>
+  </gazebo>
+  <!-- grip_link -->
+  <gazebo reference="gripper_link">
+    <kp>1000000.0</kp>
+    <kd>100.0</kd>
+    <mu1>30.0</mu1>
+    <mu2>30.0</mu2>
+    <maxVel>1.0</maxVel>
+    <minDepth>0.001</minDepth>
+    <material>Gazebo/DarkGrey</material>
+  </gazebo>
+  <!-- grip_link_sub -->
+  <gazebo reference="gripper_link_sub">
+    <kp>1000000.0</kp>
+    <kd>100.0</kd>
+    <mu1>30.0</mu1>
+    <mu2>30.0</mu2>
+    <maxVel>1.0</maxVel>
+    <minDepth>0.001</minDepth>
+    <material>Gazebo/DarkGrey</material>
   </gazebo>
   <!-- ros_control plugin -->
   <gazebo>
     <plugin name="gazebo_ros_control" filename="libgazebo_ros_control.so">
+      <robotNamespace></robotNamespace>
       <controlPeriod>0.001</controlPeriod>
       <robotSimType>gazebo_ros_control/DefaultRobotHWSim</robotSimType>
-      <legacyModeNS>true</legacyModeNS>
     </plugin>
   </gazebo>
-  <gazebo>
-    <!-- loading plugin: mimic joints works in gazebo now -->
-    <plugin name="gazebo_gripper_ros_control" filename="libroboticsgroup_gazebo_mimic_joint_plugin.so">
-      <joint>gripper</joint>
-      <mimicJoint>gripper_sub</mimicJoint>
-      <multiplier>1.0</multiplier>
-      <offset>0.0</offset>
-    </plugin>
-  </gazebo>
-  <!-- camera -->
-  <gazebo reference="camera_link">
-    <sensor type="camera" name="intel_realsense_r200">
-      <update_rate>30.0</update_rate>
-      <camera name="head">
-        <horizontal_fov>1.02974</horizontal_fov>
-        <image>
-          <width>1920</width>
-          <height>1080</height>
-          <format>R8G8B8</format>
-        </image>
-        <clip>
-          <near>0.02</near>
-          <far>300</far>
-        </clip>
-        <noise>
-          <type>gaussian</type>
-          <!-- Noise is sampled independently per pixel on each frame.
-               That pixel's noise value is added to each of its color
-               channels, which at that point lie in the range [0,1]. -->
-          <mean>0.0</mean>
-          <stddev>0.007</stddev>
-        </noise>
-      </camera>
-      <plugin name="camera_controller" filename="libgazebo_ros_camera.so">
-        <alwaysOn>true</alwaysOn>
-        <updateRate>0.0</updateRate>
-        <cameraName>camera/color</cameraName>
-        <imageTopicName>image_raw</imageTopicName>
-        <cameraInfoTopicName>camera_info</cameraInfoTopicName>
-        <frameName>camera_link</frameName>
-        <hackBaseline>0.07</hackBaseline>
-        <distortionK1>0.0</distortionK1>
-        <distortionK2>0.0</distortionK2>
-        <distortionK3>0.0</distortionK3>
-        <distortionT1>0.0</distortionT1>
-        <distortionT2>0.0</distortionT2>
-      </plugin>
-    </sensor>
-  </gazebo>
 </robot>
+<!--<?xml version="1.0"?>-->
+<!--<robot xmlns:xacro="http://ros.org/wiki/xacro">-->
+<!--  &lt;!&ndash; Gazebo Reference macro &ndash;&gt;-->
+<!--  <xacro:macro name="RefLink" params="ref">-->
+<!--    <gazebo reference="${ref}">-->
+<!--      <kp>1000000.0</kp>-->
+<!--      <kd>100.0</kd>-->
+<!--      <mu1>30.0</mu1>-->
+<!--      <mu2>30.0</mu2>-->
+<!--      <maxVel>1.0</maxVel>-->
+<!--      <minDepth>0.001</minDepth>-->
+<!--      <material>Gazebo/DarkGrey</material>-->
+<!--    </gazebo>-->
+<!--  </xacro:macro>-->
+<!--  &lt;!&ndash; World &ndash;&gt;-->
+<!--  <gazebo reference="world"/>-->
+<!--  &lt;!&ndash; Link1 &ndash;&gt;-->
+<!--  <RefLink ref="link1"/>-->
+<!--  &lt;!&ndash; Link2 &ndash;&gt;-->
+<!--  <RefLink ref="link2"/>-->
+<!--  &lt;!&ndash; Link3 &ndash;&gt;-->
+<!--  <RefLink ref="link3"/>-->
+<!--  &lt;!&ndash; Link4 &ndash;&gt;-->
+<!--  <RefLink ref="link4"/>-->
+<!--  &lt;!&ndash; Link5 &ndash;&gt;-->
+<!--  <RefLink ref="link5"/>-->
+<!--  &lt;!&ndash; gripper_link &ndash;&gt;-->
+<!--  <RefLink ref="gripper_link"/>-->
+<!--  &lt;!&ndash; gripper_link_sub &ndash;&gt;-->
+<!--  <RefLink ref="gripper_link_sub"/>-->
+<!--  &lt;!&ndash; end effector link &ndash;&gt;-->
+<!--  <gazebo reference="end_effector_link">-->
+<!--    <material>Gazebo/Red</material>-->
+<!--  </gazebo>-->
+<!--  &lt;!&ndash; ros_control plugin &ndash;&gt;-->
+<!--  <gazebo>-->
+<!--    <plugin name="gazebo_ros_control" filename="libgazebo_ros_control.so">-->
+<!--      <controlPeriod>0.001</controlPeriod>-->
+<!--      <robotSimType>gazebo_ros_control/DefaultRobotHWSim</robotSimType>-->
+<!--      <legacyModeNS>true</legacyModeNS>-->
+<!--    </plugin>-->
+<!--  </gazebo>-->
+<!--  <gazebo>-->
+<!--    <plugin name="joint_state_publisher" filename="libgazebo_ros_joint_state_publisher.so">-->
+<!--      <jointName>joint1, joint2, joint3, joint4</jointName>-->
+<!--    </plugin>-->
+<!--  </gazebo>-->
+<!--  <gazebo>-->
+<!--    &lt;!&ndash; loading plugin: mimic joints works in gazebo now &ndash;&gt;-->
+<!--    <plugin name="gazebo_gripper_ros_control" filename="libroboticsgroup_gazebo_mimic_joint_plugin.so">-->
+<!--      <joint>gripper</joint>-->
+<!--      <mimicJoint>gripper_sub</mimicJoint>-->
+<!--      <multiplier>1.0</multiplier>-->
+<!--      <offset>0.0</offset>-->
+<!--    </plugin>-->
+<!--  </gazebo>-->
+<!--  &lt;!&ndash; camera &ndash;&gt;-->
+<!--  <gazebo reference="camera_link">-->
+<!--    <sensor type="camera" name="intel_realsense_r200">-->
+<!--      <update_rate>30.0</update_rate>-->
+<!--      <camera name="head">-->
+<!--        <horizontal_fov>1.02974</horizontal_fov>-->
+<!--        <image>-->
+<!--          <width>1920</width>-->
+<!--          <height>1080</height>-->
+<!--          <format>R8G8B8</format>-->
+<!--        </image>-->
+<!--        <clip>-->
+<!--          <near>0.02</near>-->
+<!--          <far>300</far>-->
+<!--        </clip>-->
+<!--        <noise>-->
+<!--          <type>gaussian</type>-->
+<!--          &lt;!&ndash; Noise is sampled independently per pixel on each frame.-->
+<!--               That pixel's noise value is added to each of its color-->
+<!--               channels, which at that point lie in the range [0,1]. &ndash;&gt;-->
+<!--          <mean>0.0</mean>-->
+<!--          <stddev>0.007</stddev>-->
+<!--        </noise>-->
+<!--      </camera>-->
+<!--      <plugin name="camera_controller" filename="libgazebo_ros_camera.so">-->
+<!--        <alwaysOn>true</alwaysOn>-->
+<!--        <updateRate>0.0</updateRate>-->
+<!--        <cameraName>camera/color</cameraName>-->
+<!--        <imageTopicName>image_raw</imageTopicName>-->
+<!--        <cameraInfoTopicName>camera_info</cameraInfoTopicName>-->
+<!--        <frameName>camera_link</frameName>-->
+<!--        <hackBaseline>0.07</hackBaseline>-->
+<!--        <distortionK1>0.0</distortionK1>-->
+<!--        <distortionK2>0.0</distortionK2>-->
+<!--        <distortionK3>0.0</distortionK3>-->
+<!--        <distortionT1>0.0</distortionT1>-->
+<!--        <distortionT2>0.0</distortionT2>-->
+<!--      </plugin>-->
+<!--    </sensor>-->
+<!--  </gazebo>-->
+<!--</robot>-->

File: robotic_arm/urdf/open_manipulator.urdf.xacro (robot description, xacro)
@@ -2,4 +2,12 @@
 <!-- Open_Manipulator Chain -->
 <robot xmlns:xacro="http://ros.org/wiki/xacro">
+   <!-- World -->
+   <link name="world">
+   </link>
+<!-- World fixed joint -->
+   <joint name="world_fixed" type="fixed">
+     <parent link="world"/>
+     <child link="base_link"/>
+   </joint>
   <!-- Link 1 -->
   <link name="link1">
