Commit message: some bugs fixed

File: robotic_arm/urdf/robotic_arm.xacro (robot description, xacro)
@@ -1,4 +1,11 @@
 <?xml version="1.0"?>
 <robot name="robotic_arm" xmlns:xacro="http://ros.org/wiki/xacro">
+      <!-- ros_control plugin -->
+  <gazebo>
+    <plugin name="gazebo_ros_control" filename="libgazebo_ros_control.so">
+      <robotNamespace>/robotic_arm</robotNamespace>
+      <robotSimType>gazebo_ros_control/DefaultRobotHWSim</robotSimType>
+    </plugin>
+  </gazebo>
     <xacro:macro name="RefLink" params="ref">
         <gazebo reference="${ref}">
@@ -15,4 +22,5 @@
   <!--RefLink ref="world1"/ -->
   <!-- Link1 -->
+  <RefLink ref="world"/>
   <RefLink ref="link1"/>
   <!-- Link2 -->
@@ -32,5 +40,5 @@
     <material>Gazebo/Red</material>
   </gazebo>
-    <link name="world1">
+    <link name="world">
             <visual>
             <origin xyz="0 0 0" rpy="0 0 0"/>
@@ -57,13 +65,4 @@
         </inertial>
     </link>
-    <gazebo reference="world">
-          <kp>1000000.0</kp>
-          <kd>100.0</kd>
-          <mu1>30.0</mu1>
-          <mu2>30.0</mu2>
-          <maxVel>1.0</maxVel>
-          <minDepth>0.001</minDepth>
-          <material>Gazebo/Orange</material>
-    </gazebo>
     <joint name="fixed_1" type="fixed">
         <parent link="world"/>
@@ -106,5 +105,5 @@
         <origin xyz="0.012 0.0 0.017" rpy="0 0 0"/>
         <axis xyz="0 0 1"/>
-        <limit velocity="4.8" effort="1" lower="${-pi*0.9}" upper="${pi*0.9}" />
+        <limit velocity="4.8" effort="1" lower="-2.826" upper="2.826" />
     </joint>
     <!--  Link 2 -->
@@ -139,5 +138,5 @@
         <origin xyz="0.0 0.0 0.0595" rpy="0 0 0"/>
         <axis xyz="0 1 0"/>
-        <limit velocity="4.8" effort="1" lower="${-pi*0.57}" upper="${pi*0.5}" />
+        <limit velocity="4.8" effort="1" lower="-1.78" upper="1.78" />
     </joint>
     <!--  Link 3 -->
@@ -172,5 +171,5 @@
         <origin xyz="0.024 0 0.128" rpy="0 0 0"/>
         <axis xyz="0 1 0"/>
-        <limit velocity="4.8" effort="1" lower="${-pi*0.3}" upper="${pi*0.44}" />
+        <limit velocity="4.8" effort="1" lower="-0.942" upper="1.38" />
     </joint>
     <!--  Link 4 -->
@@ -205,5 +204,5 @@
         <origin xyz="0.124 0.0 0.0" rpy="0 0 0"/>
         <axis xyz="0 1 0"/>
-        <limit velocity="4.8" effort="1" lower="${-pi*0.57}" upper="${pi*0.65}" />
+        <limit velocity="4.8" effort="1" lower="-1.78" upper="2.04" />
     </joint>
     <!--  Link 5 -->
@@ -332,13 +331,4 @@
     </joint>
     <link name="camera_link"/>
-  <!-- ros_control plugin -->
-  <gazebo>
-    <plugin name="gazebo_ros_control" filename="libgazebo_ros_control.so">
-      <robotNamespace>/panda</robotNamespace>
-      <controlPeriod>0.001</controlPeriod>
-      <robotSimType>gazebo_ros_control/DefaultRobotHWSim</robotSimType>
-      <legacyModeNS>true</legacyModeNS>
-    </plugin>
-  </gazebo>
   <transmission name="tran1">
     <type>transmission_interface/SimpleTransmission</type>
@@ -348,15 +338,5 @@
     <actuator name="motor1">
       <hardwareInterface>hardware_interface/EffortJointInterface</hardwareInterface>
-      <mechanicalReduction>1</mechanicalReduction>
-    </actuator>
-  </transmission>
-  <transmission name="tran1">
-    <type>transmission_interface/SimpleTransmission</type>
-    <joint name="joint1">
-      <hardwareInterface>hardware_interface/EffortJointInterface</hardwareInterface>
-    </joint>
-    <actuator name="motor1">
-      <hardwareInterface>hardware_interface/EffortJointInterface</hardwareInterface>
-      <mechanicalReduction>1</mechanicalReduction>
+      <mechanicalReduction>100</mechanicalReduction>
     </actuator>
   </transmission>
@@ -368,5 +348,5 @@
     <actuator name="motor2">
       <hardwareInterface>hardware_interface/EffortJointInterface</hardwareInterface>
-      <mechanicalReduction>1</mechanicalReduction>
+      <mechanicalReduction>100</mechanicalReduction>
     </actuator>
   </transmission>
@@ -378,5 +358,5 @@
     <actuator name="motor3">
       <hardwareInterface>hardware_interface/EffortJointInterface</hardwareInterface>
-      <mechanicalReduction>1</mechanicalReduction>
+      <mechanicalReduction>10</mechanicalReduction>
     </actuator>
   </transmission>
@@ -388,7 +368,8 @@
     <actuator name="motor4">
       <hardwareInterface>hardware_interface/EffortJointInterface</hardwareInterface>
-      <mechanicalReduction>1</mechanicalReduction>
+      <mechanicalReduction>10</mechanicalReduction>
     </actuator>
   </transmission>
+<!--
     <transmission name="gripper_5">
       <type>transmission_interface/SimpleTransmission</type>
@@ -411,3 +392,4 @@
       </actuator>
    </transmission>
+-->
 </robot>

Commit message: new controller added

File: robotic_arm/urdf/robotic_arm.xacro (robot description, xacro)
@@ -6,4 +6,5 @@
       <robotNamespace>/robotic_arm</robotNamespace>
       <robotSimType>gazebo_ros_control/DefaultRobotHWSim</robotSimType>
+      <legacyModeNS>true</legacyModeNS>
     </plugin>
   </gazebo>
@@ -22,5 +23,5 @@
   <!--RefLink ref="world1"/ -->
   <!-- Link1 -->
-  <RefLink ref="world"/>
+  <!--RefLink ref="base_link"/-->
   <RefLink ref="link1"/>
   <!-- Link2 -->
@@ -40,33 +41,48 @@
     <material>Gazebo/Red</material>
   </gazebo>
-    <link name="world">
-            <visual>
-            <origin xyz="0 0 0" rpy="0 0 0"/>
-            <geometry>
-               <box size="0.5 0.5 0.05"/>
-            </geometry>
-            <material name="green">
-                <color rgba="0.0 0.8 0.0 1.0"/>
-            </material>
-        </visual>
-        <collision>
-            <origin xyz="0 0 0" rpy="0 0 0"/>
-            <geometry>
-                <box size="0.5 0.5 0.05"/>
-            </geometry>
-        </collision>
-        <inertial>
-          <origin xyz="0 0 0" rpy="0 0 0"/>
-          <mass value="1"/>
-          <inertia
-            ixx="1.0" ixy="0.0" ixz="0.0"
-            iyy="1.0" iyz="0.0"
-            izz="1.0"/>
-        </inertial>
-    </link>
-    <joint name="fixed_1" type="fixed">
-        <parent link="world"/>
-        <child link="link1"/>
-    </joint>
+<!--  <gazebo reference="robot_base">-->
+<!--    <kp>1000000.0</kp>-->
+<!--    <kd>100.0</kd>-->
+<!--    <mu1>30.0</mu1>-->
+<!--    <mu2>30.0</mu2>-->
+<!--    <maxVel>1.0</maxVel>-->
+<!--    <minDepth>0.001</minDepth>-->
+<!--    <material>Gazebo/Orange</material>-->
+<!--  </gazebo>-->
+  <link name="world" />
+  <joint name="world_joint" type="fixed">
+    <parent link="world" />
+    <child link = "link1" />
+    <origin xyz="0.0 0.0 0.0" rpy="0.0 0.0 0.0" />
+  </joint>
+<!--    <link name="base_link">-->
+<!--            <visual>-->
+<!--            <origin xyz="0 0 0" rpy="0 0 0"/>-->
+<!--            <geometry>-->
+<!--               <box size="0.5 0.5 0.07"/>-->
+<!--            </geometry>-->
+<!--            <material name="green">-->
+<!--                <color rgba="0.0 0.8 0.0 1.0"/>-->
+<!--            </material>-->
+<!--        </visual>-->
+<!--        <collision>-->
+<!--            <origin xyz="0 0 0" rpy="0 0 0"/>-->
+<!--            <geometry>-->
+<!--                <box size="0.5 0.5 0.07"/>-->
+<!--            </geometry>-->
+<!--        </collision>-->
+<!--        <inertial>-->
+<!--          <origin xyz="0 0 0" rpy="0 0 0"/>-->
+<!--          <mass value="1"/>-->
+<!--          <inertia-->
+<!--            ixx="1.0" ixy="0.0" ixz="0.0"-->
+<!--            iyy="1.0" iyz="0.0"-->
+<!--            izz="1.0"/>-->
+<!--        </inertial>-->
+<!--    </link>-->
+<!--    <joint name="fixed_1" type="fixed">-->
+<!--        <parent link="world"/>-->
+<!--        <child link="link1"/>-->
+<!--    </joint>-->
     <!-- Link 1 -->
     <link name="link1">
@@ -125,5 +141,5 @@
         </collision>
         <inertial>
-            <origin xyz="-3.0184870e-04 5.4043684e-04 ${0.018 + 2.9433464e-02}" />
+            <origin xyz="-3.0184870e-04 5.4043684e-04 0.047433464" />
             <mass value="9.8406837e-02"/>
             <inertia ixx="3.4543422e-05" ixy="-1.6031095e-08" ixz="-3.8375155e-07"

Commit message: edited

File: robotic_arm/urdf/robotic_arm.xacro (robot description, xacro)
@@ -20,8 +20,4 @@
         </gazebo>
     </xacro:macro>
-  <!-- World -->
-  <!--RefLink ref="world1"/ -->
-  <!-- Link1 -->
-  <!--RefLink ref="base_link"/-->
   <RefLink ref="link1"/>
   <!-- Link2 -->
@@ -41,13 +37,4 @@
     <material>Gazebo/Red</material>
   </gazebo>
-<!--  <gazebo reference="robot_base">-->
-<!--    <kp>1000000.0</kp>-->
-<!--    <kd>100.0</kd>-->
-<!--    <mu1>30.0</mu1>-->
-<!--    <mu2>30.0</mu2>-->
-<!--    <maxVel>1.0</maxVel>-->
-<!--    <minDepth>0.001</minDepth>-->
-<!--    <material>Gazebo/Orange</material>-->
-<!--  </gazebo>-->
   <link name="world" />
   <joint name="world_joint" type="fixed">
@@ -56,33 +43,4 @@
     <origin xyz="0.0 0.0 0.0" rpy="0.0 0.0 0.0" />
   </joint>
-<!--    <link name="base_link">-->
-<!--            <visual>-->
-<!--            <origin xyz="0 0 0" rpy="0 0 0"/>-->
-<!--            <geometry>-->
-<!--               <box size="0.5 0.5 0.07"/>-->
-<!--            </geometry>-->
-<!--            <material name="green">-->
-<!--                <color rgba="0.0 0.8 0.0 1.0"/>-->
-<!--            </material>-->
-<!--        </visual>-->
-<!--        <collision>-->
-<!--            <origin xyz="0 0 0" rpy="0 0 0"/>-->
-<!--            <geometry>-->
-<!--                <box size="0.5 0.5 0.07"/>-->
-<!--            </geometry>-->
-<!--        </collision>-->
-<!--        <inertial>-->
-<!--          <origin xyz="0 0 0" rpy="0 0 0"/>-->
-<!--          <mass value="1"/>-->
-<!--          <inertia-->
-<!--            ixx="1.0" ixy="0.0" ixz="0.0"-->
-<!--            iyy="1.0" iyz="0.0"-->
-<!--            izz="1.0"/>-->
-<!--        </inertial>-->
-<!--    </link>-->
-<!--    <joint name="fixed_1" type="fixed">-->
-<!--        <parent link="world"/>-->
-<!--        <child link="link1"/>-->
-<!--    </joint>-->
     <!-- Link 1 -->
     <link name="link1">
@@ -110,9 +68,4 @@
         </inertial>
     </link>
-        <!-- Joint 0 -->
-<!--    <joint name="joint0" type="fixed">
-        <parent link="world"/>
-        <child link="link1"/>
-    </joint>-->
     <!-- Joint 1 -->
     <joint name="joint1" type="revolute">
@@ -387,25 +340,23 @@
     </actuator>
   </transmission>
-<!--
-    <transmission name="gripper_5">
-      <type>transmission_interface/SimpleTransmission</type>
-      <joint name="gripper">
-        <hardwareInterface>hardware_interface/EffortJointInterface</hardwareInterface>
-      </joint>
-      <actuator name="gripper_motor">
-        <mechanicalReduction>1</mechanicalReduction>
-        <hardwareInterface>hardware_interface/EffortJointInterface</hardwareInterface>
-      </actuator>
-   </transmission>
-    <transmission name="gripper_sub_6">
-      <type>transmission_interface/SimpleTransmission</type>
-      <joint name="gripper_sub">
-        <hardwareInterface>hardware_interface/EffortJointInterface</hardwareInterface>
-      </joint>
-      <actuator name="gripper_sub_motor">
-        <mechanicalReduction>1</mechanicalReduction>
-        <hardwareInterface>hardware_interface/EffortJointInterface</hardwareInterface>
-      </actuator>
-   </transmission>
--->
+<!--    <transmission name="gripper_5">-->
+<!--      <type>transmission_interface/SimpleTransmission</type>-->
+<!--      <joint name="gripper">-->
+<!--        <hardwareInterface>hardware_interface/EffortJointInterface</hardwareInterface>-->
+<!--      </joint>-->
+<!--      <actuator name="gripper_motor">-->
+<!--        <mechanicalReduction>1</mechanicalReduction>-->
+<!--        <hardwareInterface>hardware_interface/EffortJointInterface</hardwareInterface>-->
+<!--      </actuator>-->
+<!--   </transmission>-->
+<!--    <transmission name="gripper_sub_6">-->
+<!--      <type>transmission_interface/SimpleTransmission</type>-->
+<!--      <joint name="gripper_sub">-->
+<!--        <hardwareInterface>hardware_interface/EffortJointInterface</hardwareInterface>-->
+<!--      </joint>-->
+<!--      <actuator name="gripper_sub_motor">-->
+<!--        <mechanicalReduction>1</mechanicalReduction>-->
+<!--        <hardwareInterface>hardware_interface/EffortJointInterface</hardwareInterface>-->
+<!--      </actuator>-->
+<!--   </transmission>-->
 </robot>
